Commit message: Stashed newer updates

File: urdf/asv_controllers.xacro (robot description, xacro)
@@ -3,6 +3,6 @@
 <transmission name="left_thruster_rotation">
   <type>transmission_interface/SimpleTransmission</type>
-  <joint name="body_to_thruster_left">
-    <hardwareInterface>hardware_interface/EffortJointInterface</hardwareInterface>
+  <joint name="left_thruster_to_prop">
+    <hardwareInterface>hardware_interface/VelocityJointInterface</hardwareInterface>
   </joint>
   <actuator name="left_thruster_actuator">
@@ -12,6 +12,6 @@
 <transmission name="right_thruster_rotation">
   <type>transmission_interface/SimpleTransmission</type>
-  <joint name="body_to_thruster_right">
-    <hardwareInterface>hardware_interface/EffortJointInterface</hardwareInterface>
+  <joint name="right_thruster_to_prop">
+    <hardwareInterface>hardware_interface/VelocityJointInterface</hardwareInterface>
   </joint>
   <actuator name="right_thruster_actuator">
